File: PIM_V02/PIM_V02.kicad_pcb (KiCad board)
At the start: 4 copper layers, 93 x 62 mm, 260 parts, among them J1 Conn_01x06, J10 Conn_02x08_Odd_Even, J11 Conn_01x02, J12 Conn_01x02, J13 Conn_01x02, J4 USB_C_Receptacle_USB2.0_14P, J5 Conn_01x04, J6 Conn_01x04, J7 Conn_02x03_Odd_Even, J8 Conn_01x02, J9 Conn_02x08_Odd_Even, Q1 SQJ407EP-T1_GE3, Q2 PMOS, Q3 PMOS, Q4 NMOS, SW1 SW_Push, U1 TPS259541DSGR, U10 TPS62933, U11 AP2112K-3.3, U12 MP28167GQ-A-P, U13 GD5F1GQ5UEYIGR, U14 MB85RS256B, U2 USBLC6-2SC6, U3 STM32H7A3VITx, U4 MCP2562FDT-E/SN, U5 MCP2562FDT-E/SN, U6 TPS62933, U7 TPS62933, U8 TPS62933, U9 TPS62933, Y1 Crystal_GND24_Small

Commit message: more changes, near final schematic and part way through layout now
Parts:
- removed J7: Conn_02x03_Odd_Even, Connector_PinHeader_2.54mm:PinHeader_2x03_P2.54mm_Vertical
- added C109: 0.1uF, Capacitor_SMD:C_0603_1608Metric, F.Cu at (190.3, 92.1)
- added C111: 4.7uF, Capacitor_SMD:C_0603_1608Metric, F.Cu at (148.4, 40.6)
- added C112: 0.1uF, Capacitor_SMD:C_0603_1608Metric, F.Cu at (161.4, 41.7)
- added C113: 0.1uF, Capacitor_SMD:C_0603_1608Metric, F.Cu at (148.4, 42.1)
- added C114: 0.1uF, Capacitor_SMD:C_0603_1608Metric, F.Cu at (161.4, 43.3)
- added C115: 0.1uF, Capacitor_SMD:C_0603_1608Metric, F.Cu at (148.4, 37.6)
- added C116: 0.1uF, Capacitor_SMD:C_0603_1608Metric, F.Cu at (157.6, 47.9)
- added C117: 0.1uF, Capacitor_SMD:C_0603_1608Metric, F.Cu at (161.4, 39.7)
- added Q5: 2N7002, Package_TO_SOT_SMD:SOT-23, B.Cu at (96.9, 109.4)
- added R100: 33R, Resistor_SMD:R_0603_1608Metric, F.Cu at (144.2, 41.7)
- added R101: 10kR, Resistor_SMD:R_0603_1608Metric, F.Cu at (148.8, 47.2)
- added R102: 33R, Resistor_SMD:R_0603_1608Metric, F.Cu at (165.8, 36.7)
- added R103: 33R, Resistor_SMD:R_0603_1608Metric, F.Cu at (165.8, 38.2)
- added R104: 33R, Resistor_SMD:R_0603_1608Metric, F.Cu at (165.8, 39.7)
- added R105: 33R, Resistor_SMD:R_0603_1608Metric, F.Cu at (165.8, 41.2)
- added R106: 33R, Resistor_SMD:R_0603_1608Metric, F.Cu at (165.8, 42.7)
- added R107: 33R, Resistor_SMD:R_0603_1608Metric, F.Cu at (165.8, 44.4)
- added R108: 33R, Resistor_SMD:R_0603_1608Metric, F.Cu at (165.8, 45.9)
- added R109: 33R, Resistor_SMD:R_0603_1608Metric, F.Cu at (165.8, 47.4)
- added R110: 4.7kR, Resistor_SMD:R_0603_1608Metric, F.Cu at (169.3, 36.7)
- added R111: 4.7kR, Resistor_SMD:R_0603_1608Metric, F.Cu at (169.3, 38.2)
- added R112: 4.7kR, Resistor_SMD:R_0603_1608Metric, F.Cu at (169.3, 39.7)
- added R113: 4.7kR, Resistor_SMD:R_0603_1608Metric, F.Cu at (169.3, 41.2)
- added R114: 4.7kR, Resistor_SMD:R_0603_1608Metric, F.Cu at (169.3, 42.7)
- added R115: 4.7kR, Resistor_SMD:R_0603_1608Metric, F.Cu at (169.3, 44.4)
- added R116: 4.7kR, Resistor_SMD:R_0603_1608Metric, F.Cu at (169.3, 45.9)
- added R117: 4.7kR, Resistor_SMD:R_0603_1608Metric, F.Cu at (169.3, 47.4)
- added R118: 33R, Resistor_SMD:R_0603_1608Metric, F.Cu at (144.2, 43.2)
- added R119: 33R, Resistor_SMD:R_0603_1608Metric, F.Cu at (144.2, 44.7)
- added R120: 33R, Resistor_SMD:R_0603_1608Metric, F.Cu at (144.2, 46.2)
- added R121: 33R, Resistor_SMD:R_0603_1608Metric, F.Cu at (144.2, 47.7)
- added R122: 33R, Resistor_SMD:R_0603_1608Metric, F.Cu at (157.6, 34.9)
- added R123: 4.7kR, Resistor_SMD:R_0603_1608Metric, F.Cu at (157.6, 31.9)
- added R124: 4.7kR, Resistor_SMD:R_0603_1608Metric, F.Cu at (140.5, 43.2)
- added R125: 4.7kR, Resistor_SMD:R_0603_1608Metric, F.Cu at (140.5, 44.7)
- added R126: 4.7kR, Resistor_SMD:R_0603_1608Metric, F.Cu at (140.5, 46.2)
- added R127: 4.7kR, Resistor_SMD:R_0603_1608Metric, F.Cu at (140.5, 47.7)
- added R87: 1k, Resistor_SMD:R_0603_1608Metric, B.Cu at (93.3, 110.3)
- added R88: 100k, Resistor_SMD:R_0603_1608Metric, B.Cu at (99.4, 110.8)
- added R89: 10R, Resistor_SMD:R_0603_1608Metric, F.Cu at (190.3, 94.6)
- added R90: 100R, Resistor_SMD:R_0603_1608Metric, F.Cu at (172.6, 42.2)
- added R91: 10mR, Resistor_SMD:R_0603_1608Metric, B.Cu at (168.9, 90.2)
- added R92: 10mR, Resistor_SMD:R_0603_1608Metric, F.Cu at (190.3, 99.6)
- added R93: 10mR, Resistor_SMD:R_0603_1608Metric, F.Cu at (190.3, 102.1)
- added R94: 10R, Resistor_SMD:R_0603_1608Metric, F.Cu at (194.4, 89.5)
- added R95: 10R, Resistor_SMD:R_0603_1608Metric, F.Cu at (194.4, 92.1)
- added R96: 10R, Resistor_SMD:R_0603_1608Metric, F.Cu at (194.4, 94.6)
- added R97: 10R, Resistor_SMD:R_0603_1608Metric, F.Cu at (194.4, 97.1)
- added R98: 10R, Resistor_SMD:R_0603_1608Metric, F.Cu at (194.4, 99.6)
- added R99: 33R, Resistor_SMD:R_0603_1608Metric, F.Cu at (152.6, 48.2)
- added TP10: TestPoint, TestPoint:TestPoint_Pad_D1.0mm, F.Cu at (160.5, 47.3)
- added TP11: TestPoint, TestPoint:TestPoint_Pad_D1.0mm, F.Cu at (152.6, 50.8)
- added TP12: TestPoint, TestPoint:TestPoint_Pad_D1.0mm, F.Cu at (154.4, 47.6)
- added TP13: TestPoint, TestPoint:TestPoint_Pad_D1.0mm, F.Cu at (154.5, 49.8)
- added TP14: TestPoint, TestPoint:TestPoint_Pad_D1.0mm, F.Cu at (154.1, 52.3)
- added TP15: TestPoint, TestPoint:TestPoint_Pad_D1.0mm, F.Cu at (148.8, 44.6)
- added TP16: TestPoint, TestPoint:TestPoint_Pad_D1.0mm, F.Cu at (142.0, 39.5)
- added TP17: TestPoint, TestPoint:TestPoint_Pad_D1.0mm, F.Cu at (150.5, 35.2)
- added TP18: TestPoint, TestPoint:TestPoint_Pad_D1.0mm, F.Cu at (144.5, 38.7)
- added TP19: TestPoint, TestPoint:TestPoint_Pad_D1.0mm, F.Cu at (110.1, 86.7)
- added TP20: TestPoint, TestPoint:TestPoint_Pad_D1.0mm, F.Cu at (108.3, 82.9)
- added TP22: TestPoint, TestPoint:TestPoint_Pad_D1.0mm, F.Cu at (108.5, 79.2)
- added TP23: TestPoint, TestPoint:TestPoint_Pad_D1.0mm, F.Cu at (112.6, 86.2)
- added TP24: TestPoint, TestPoint:TestPoint_Pad_D1.0mm, F.Cu at (119.6, 87.2)
- added TP9: TestPoint, TestPoint:TestPoint_Pad_D1.0mm, F.Cu at (160.7, 45.2)
- added U15: ICE40UP5K-SG48I, ICE40UP5K-SG48I:QFN48_L-ASC10_ICE40ULTRAPLUS_MACHXO2_LAT, F.Cu at (154.8, 41.4)
- added U16: INA3221, Package_DFN_QFN:Texas_RGV0016A_VQFN-16-1EP_4x4mm_P0.65mm_EP2.1x2.1mm, F.Cu at (191.7, 82.2)
- C1, C104, C72, C8, C80, C95, C99: value C_Small -> 1uF
- C10, C11, C14, C15, C94: value C_Small -> 4.7uF
- C100, C64: value C_Small -> 27pF
- C101, C102, C68, C69, C75, C76, C77: value C_Small -> 22uF; footprint Capacitor_SMD:C_0603_1608Metric -> Capacitor_SMD:C_0805_2012Metric
- C103, C12, C13, C16, C17, C2, C34, C36, C40, C41, C42, C53, C54, C57, C58, C70, C73, C74, C81, C83, C84, C85, C86, C87, C88, C89, C90, C91, C92, C93, C98: value C_Small -> 0.1uF
- C105, C106, C107, C108, C38, C55, C56, C65, C66, C67: value C_Small -> 10nF
- C18, C19, C20, C21, C22, C23, C24, C25: value C_Small -> 47pF
- C26, C27: value C_Small -> 4.7nF
- C28, C29, C30, C31, C32, C33, C49, C50, C51, C52, C9: value C_Small -> 10uF
- C3: value C_Small -> 3.3nF
- C35: value C_Small -> 0.1uF; moved to F.Cu
- C37, C39: value C_Small -> 33nF
- C4, C5: value C_Small -> 47uF; footprint Capacitor_SMD:C_0603_1608Metric -> Capacitor_SMD:C_1206_3216Metric; moved to B.Cu
- C43, C44, C45, C46, C47, C48, C59, C60, C61, C62: value C_Small -> 22uF
- C6, C7, C82: value C_Small -> 10uF; moved to B.Cu
- C63: value C_Small -> 100nF
- C71: value C_Small -> 22nF
- C78, C79: value C_Small -> 1uF; moved to B.Cu
- C96, C97: value C_Small -> 2.2uF
- D1: value SMBJ12A -> SMBJ13A; footprint CustomFootprints:SMBJ12A -> CustomFootprints:SMBJ13A; moved to B.Cu
- D13: value SMBJ12A -> SMBJ13A; footprint CustomFootprints:SMBJ12A -> CustomFootprints:SMBJ13A
- D3: value D_Schottky -> PMEG4010
- D4: value D_Zener -> BZT52C15; moved to B.Cu
- FL1, FL2: value ACT45B-101-2P-TL003 -> Choke_CommonMode_FerriteCore_1243; footprint CustomFootprints:ACT45B-101-2P-TL003_TDK -> Inductor_SMD:L_CommonModeChoke_Coilcraft_1812CAN
- L1, L2, L3, L4, L5: value L_Small -> 6.8uH
- L6: value L_Small -> 4.7uH
- Q1, U11, U2: moved to B.Cu
- R1, R4: value R_Small -> 5k1R; moved to B.Cu
- R10, R11, R16, R17, R22, R23, R24, R35, R36, R74, R75, R76, R77, R78, R83, R84, R85, R86, R9: value R_Small -> 0R
- R12, R69: value R_Small -> 1MR
- R13, R14, R15, R26, R28, R30, R38, R40, R59, R60, R61, R66, R67, R7: value R_Small -> 10kR
- R18, R19, R20, R21: value R_Small -> 60R
- R2: value R_Small -> 866kR
- R25, R37: value R_Small -> 52.3kR
- R27, R39: value R_Small -> 31.6kR
- R29: value R_Small -> 4.99kR
- R3: value R_Small -> 150kR
- R31, R33, R6: value R_Small -> 470R
- R32, R34, R81, R82: value R_Small -> 100R
- R41, R42, R43, R44: value R_Small -> 1kR
- R45, R47, R49: value R_Small -> 470kR
- R46, R48, R50, R68, R70, R71, R72, R73: value R_Small -> 100kR
- R5: value R_Small -> 511R
- R51, R52, R57, R58: value R_Small -> 4.7kR
- R53: value R_Small -> 430kR
- R54: value R_Small -> 400kR
- R55: value R_Small -> 21.5kR
- R56: value R_Small -> 43.2kR
- R62, R63, R64, R65: value R_Small -> 33R
- R79, R80: value R_Small -> 1.8kR
- R8: value R_Small -> 100kR; moved to B.Cu
- U13: value GD5F1GQ5UEYIGR -> MT29F1G01ABAFDWB-IT_F
- moved J9 107.7 mm to (223.5, 39.9), turned to 0 degrees
- moved C35 78.2 mm to (190.3, 89.5)
- moved C103 51.0 mm to (101.2, 63.7)
- moved R66 44.4 mm to (156.8, 51.0), turned to 180 degrees
- moved C104 42.6 mm to (111.1, 62.4)
- moved R67 41.8 mm to (139.9, 41.4)
- moved U14 41.6 mm to (106.2, 63.9)
- moved C1 40.0 mm to (96.1, 101.9)
- moved C8 40.0 mm to (102.9, 100.7)
- moved D3 40.0 mm to (101.0, 99.6)
- moved R2 40.0 mm to (97.2, 104.2)
- moved R3 40.0 mm to (97.2, 105.7)
- moved R5 40.0 mm to (102.4, 106.5)
- moved R7 40.0 mm to (103.9, 106.5)
- moved C2 40.0 mm to (97.8, 101.9)
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Connections:
- net /VARI_SCL renamed /POWER_SCL
- net /VARI_SDA renamed /POWER_SDA
- net Net-(U1-EN_UVLO) renamed /EFUSE_ENxxx
- C101 pad 1: +VARI_PL -> /POWER/SUP_VARI_PL
- C102 pad 1: +VARI_PL -> /POWER/SUP_VARI_PL
- C59 pad 1: +5V_PL -> /POWER/SUP_5V_PL
- C60 pad 1: +3V3_PL -> /POWER/SUP_3V3_PL
- C61 pad 1: +5V_PL -> /POWER/SUP_5V_PL
- C62 pad 1: +3V3_PL -> /POWER/SUP_3V3_PL
- C75 pad 1: +VARI_PL -> /POWER/SUP_VARI_PL
- C76 pad 1: +VARI_PL -> /POWER/SUP_VARI_PL
- C77 pad 1: +VARI_PL -> /POWER/SUP_VARI_PL
- C86 pad 1: +5V_PL -> /POWER/SUP_5V_PL
- C87 pad 1: +3V3_PL -> /POWER/SUP_3V3_PL
- C88 pad 1: +VARI_PL -> /POWER/SUP_VARI_PL
- FL1 pad 1: /CAN/CAN0_RAW_P -> /CAN/CAN0_RAW_N
- FL1 pad 2: /CAN/CAN0_RAW_N -> /CAN0_N
- FL1 pad 3: /CAN0_N -> /CAN0_P
- FL1 pad 4: /CAN0_P -> /CAN/CAN0_RAW_P
- FL2 pad 1: /CAN/CAN1_RAW_P -> /CAN/CAN1_RAW_N
- FL2 pad 2: /CAN/CAN1_RAW_N -> /CAN1_N
- FL2 pad 3: /CAN1_N -> /CAN1_P
- FL2 pad 4: /CAN1_P -> /CAN/CAN1_RAW_P
- L4 pad 2: +5V_PL -> /POWER/SUP_5V_PL
- L5 pad 2: +3V3_PL -> /POWER/SUP_3V3_PL
- R37 pad 1: +5V_PL -> /POWER/SUP_5V_PL
- R39 pad 1: +3V3_PL -> /POWER/SUP_3V3_PL
- R53 pad 2: +VARI_PL -> /POWER/SUP_VARI_PL
- R64 pad 1: /nSS_SPI_FPGA -> Net-(U3-PA4)
- R64 pad 2: Net-(U3-PD11) -> /nSS_SPI_FPGA
- R65 pad 1: /nCRESET_FPGA -> Net-(U3-PC4)
- R65 pad 2: Net-(U3-PD12) -> /nCRESET_FPGA
- R66 pad 1: +3V3_MCU -> +3V3_HK
- R67 pad 1: +3V3_MCU -> +3V3_HK
- R7 pad 1: +3V3_HK -> +3V3_MCU
- R7 pad 2: /PL_FLT -> /nPL_FLT
- U1 pad 6: /PL_FLT -> /nPL_FLT
- U12 pad 12: +VARI_PL -> /POWER/SUP_VARI_PL
- U13 pad 9: GND -> (no net)
- U3 pad 28: unconnected-(U3-PA4-Pad28) -> Net-(U3-PA4)
- U3 pad 32: unconnected-(U3-PC4-Pad32) -> Net-(U3-PC4)
- U3 pad 33: unconnected-(U3-PC5-Pad33) -> /CDONE_FPGA
- U3 pad 34: unconnected-(U3-PB0-Pad34) -> /FPGA_INT
- U3 pad 35: unconnected-(U3-PB1-Pad35) -> /FPGA_EXTRA
- U3 pad 58: Net-(U3-PD11) -> unconnected-(U3-PD11-Pad58)
- U3 pad 59: Net-(U3-PD12) -> unconnected-(U3-PD12-Pad59)
- U3 pad 60: /CDONE_FPGA -> unconnected-(U3-PD13-Pad60)
- U3 pad 61: /FPGA_INT -> unconnected-(U3-PD14-Pad61)
- U3 pad 62: /FPGA_EXTRA -> unconnected-(U3-PD15-Pad62)
- U3 pad 86: unconnected-(U3-PD5-Pad86) -> /nPL_FLT
- U3 pad 87: unconnected-(U3-PD6-Pad87) -> /EFUSE_EN
Routing:
- net /USART3_TX_PL: track 59.1 -> 4.21 mm, vias 1 -> 0
- net /USART3_RX_PL: track 55.5 -> 5.87 mm, vias 1 -> 0
- net /SPI2_SCK_PL: track 51.3 -> 2.12 mm, vias 1 -> 0
- net /I2C2_SDA_PL: track 63.3 -> 15.3 mm, vias 2 -> 1
- net /SPI2_MISO_PL: track 50.0 -> 2.44 mm, vias 2 -> 1
- net /SPI2_MOSI_PL: track 49.1 -> 2.38 mm, vias 2 -> 1
- net /I2C2_SCL_PL: track 59.4 -> 16.3 mm, vias 1 -> 0
- net +3V3_HK: track 107.4 -> 67.0 mm, vias 8 -> 6
- net /OCTOSPI1_BK2_NCS: track 40.1 -> 2.61 mm
- net /CDONE_FPGA: track 35.1 -> 0.00 mm, vias 1 -> 0
- net /OCTOSPI1_BK2_IO2: track 41.9 -> 7.40 mm
- net /POWER_SDA: track 37.6 -> 5.37 mm, vias 1 -> 0
- net /POWER_SCL: track 34.9 -> 4.85 mm, vias 1 -> 0
- net /OCTOSPI1_BK2_IO1: track 37.7 -> 7.70 mm
- net /FPGA_EXTRA: track 29.9 -> 0.00 mm, vias 1 -> 0
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- added copper zone on B.Cu, net +12V_IN
- added copper zone on B.Cu, net /POWER/SUP_5V_PL
- removed copper zone on F.Cu, net +12V_HK
- removed copper zone on B.Cu, net +5V_PL
Other:
- board text added: "VARI RAIL ON BOT (BC MCU)"
- board text removed: "CAN1_N"
- board text removed: "CAN1_P"
