File: PIM_V02/PIM_V02.kicad_pcb (KiCad board)
At the start: 4 copper layers, 95.9 x 90.2 mm, 369 parts, among them J1 Conn_01x06, J10 Conn_01x06, J11 Conn_01x06, J12 Conn_01x12, J13 Conn_01x12, J14 Conn_01x04, J4 USB_C_Receptacle_USB2.0_14P, J5 Conn_01x04, J6 Conn_01x04, J9 Conn_01x06, Q1 SQJ407EP-T1_GE3, Q2 PMOS, Q3 PMOS, Q4 NMOS, SW1 SW_Push, U1 TPS259540DSGR, U10 TPS62933, U11 AP2112K-3.3, U12 MP28167GQ-A-P, U13 MT29F1G01ABAFDWB-IT_F, U14 MB85RS256B, U15 ICE40UP5K-SG48I, U16 INA3221, U17 MCP2518FDT-E/SL, U18 MCP2562FDT-E/SN, U2 USBLC6-2SC6, U3 STM32H7A3VITx, U4 MCP2562FDT-E/SN, U5 MCP2562FDT-E/SN, U6 TPS62933, U7 TPS62933, U8 TPS62933, U9 TPS62933, Y1 Crystal_GND24_Small, Y2 Crystal_GND24_Small

Commit message: No errors, just need to clean up the silkscreen. ready for a review
Parts:
- moved C46 1.95 mm to (125.4, 107.9)
- moved C83 1.95 mm to (123.9, 107.9)
- moved C59 1.75 mm to (148.4, 70.6)
- moved C86 1.75 mm to (146.9, 70.6)
- moved C60 1.66 mm to (148.4, 86.8)
- moved C87 1.66 mm to (146.9, 86.8)
- moved C62 1.56 mm to (147.1, 91.6)
- moved C43 1.40 mm to (124.3, 101.9)
- moved R31 1.30 mm to (125.9, 102.0)
- moved R136 1.22 mm to (127.6, 103.6)
- moved R137 1.12 mm to (129.2, 103.6)
- moved C68 1.04 mm to (131.0, 101.9)
- moved R59 0.60 mm to (119.6, 60.7)
- moved C45 0.58 mm to (124.3, 86.2)
- moved R130 0.50 mm to (111.3, 80.7)
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Connections:
- R59 pad 1: unconnected-(R59-Pad1) -> +3V3_MCU
- R59 pad 2: unconnected-(R59-Pad2) -> /OCTOSPI1_BK2_NCS
Routing:
- net GND: track 4.89 -> 14.1 mm, vias 96 -> 244
- net /POWER/SUP_5V_PL: track 28.2 -> 35.7 mm
- net +3V3_MCU: track 113.1 -> 106.9 mm, vias 33 -> 29
- net +5V_HK: track 78.2 -> 80.9 mm
- net /+VARI_EN: track 28.6 -> 27.0 mm
- net +3V3_HK: track 137.5 -> 139.1 mm, vias 31 -> 30
- net /SPI1_SCK_FPGA: track 81.9 -> 82.9 mm
- net /SPI_SCK_CAN2: track 85.8 -> 86.8 mm
- net /POWER/SUP_3V3_PL: track 58.9 -> 57.9 mm
- net /nSS_SPI_FPGA: track 82.1 -> 83.1 mm
- net /POWER_SCL: track 92.8 -> 91.8 mm
- net Net-(D9-A): track 1.39 -> 2.33 mm
- net +5V_PL: track 96.4 -> 97.1 mm
- net /POWER_SDA: track 86.8 -> 86.2 mm, vias 4 -> 2
- net /EN_EF: vias 4 -> 3
