File: PIM_V02/POWER.kicad_sch (KiCad schematic)
At the start: 114 parts, among them J11 Conn_01x02, J12 Conn_01x02, J13 Conn_01x02, U10 TPS62933, U12 MP28167GQ-A-P, U6 TPS62933, U7 TPS62933, U8 TPS62933, U9 TPS62933

Commit message: more changes, near final schematic and part way through layout now
Parts:
- added C109: 0.1uF, Capacitor_SMD:C_0603_1608Metric, symbol Device:C_Small
- added R89, R94, R95, R96, R97, R98: 10R, Resistor_SMD:R_0603_1608Metric, symbol Device:R_Small
- added R91, R92, R93: 10mR, Resistor_SMD:R_0603_1608Metric, symbol Device:R_Small
- added U16: INA3221, Package_DFN_QFN:Texas_RGV0016A_VQFN-16-1EP_4x4mm_P0.65mm_EP2.1x2.1mm, symbol Power_Management:INA3221
- C101, C102, C76, C77: value C_Small -> 22uF; footprint Capacitor_SMD:C_0603_1608Metric -> Capacitor_SMD:C_0805_2012Metric; MPN GRT188R61A226ME13D -> GRM21BR61E226ME44L; PD CAP CER 22UF 10V X5R 0603 -> CAP CER 22UF 25V X5R 0805
- C28, C29, C30, C31, C32, C33, C49, C50, C51, C52: value C_Small -> 10uF
- C34, C35, C36, C40, C41, C42, C53, C54, C57, C58, C70, C73, C74, C83, C84, C85, C86, C87, C88: value C_Small -> 0.1uF
- C37, C39: value C_Small -> 33nF
- C38, C55, C56, C65, C66, C67: value C_Small -> 10nF
- C43, C44, C45, C46, C47, C48, C59, C60, C61, C62: value C_Small -> 22uF
- C68, C75: value C_Small -> 22uF; footprint Capacitor_SMD:C_0603_1608Metric -> Capacitor_SMD:C_0805_2012Metric; MPN GRT188R61E106ME13D -> GRM21BR61E226ME44L; Note 10uF for dev -> (none); PD CAP CER 10UF 25V X5R 0603 -> CAP CER 22UF 25V X5R 0805
- C69: value C_Small -> 22uF; footprint Capacitor_SMD:C_0603_1608Metric -> Capacitor_SMD:C_0805_2012Metric; MPN GRT188R61E106ME13D -> GRM21BR61E226ME44L; PD CAP CER 10UF 25V X5R 0603 -> CAP CER 22UF 25V X5R 0805
- C71: value C_Small -> 22nF
- C72: value C_Small -> 1uF
- L1, L2, L3, L4, L5: value L_Small -> 6.8uH
- L6: value L_Small -> 4.7uH
- R10, R22, R23, R24, R35, R36, R74, R75, R76, R77, R78, R9: value R_Small -> 0R
- R25, R37: value R_Small -> 52.3kR
- R26, R28, R30, R38, R40: value R_Small -> 10kR
- R27, R39: value R_Small -> 31.6kR
- R29: value R_Small -> 4.99kR
- R31, R33: value R_Small -> 470R
- R32, R34: value R_Small -> 100R
- R45, R47, R49: value R_Small -> 470kR
- R46, R48, R50, R71, R72, R73: value R_Small -> 100kR
- R53: value R_Small -> 430kR
- R54: value R_Small -> 400kR
- R55: value R_Small -> 21.5kR
- R56: value R_Small -> 43.2kR
Connections:
- net +3V3_PL: now also R92.2, R96.1; no longer C60.1, C62.1, C87.1, L5.2, R39.1
- net +5V_PL: now also R91.2, R94.1; no longer C59.1, C61.1, C86.1, L4.2, R37.1
- net +VARI_PL: now also R93.2, R98.1; no longer C101.1, C102.1, C75.1, C76.1, C77.1, C88.1, R53.2, U12.12 (OUT)
- net GND: now also C109.2, U16.17 (EP), U16.3 (GND), U16.5 (A0)
- net VARI_SCL renamed POWER_SCL
- net POWER_SCL: now also U16.6 (SCL)
- net VARI_SDA renamed POWER_SDA
- net POWER_SDA: now also U16.7 (SDA)
- new net: R98.2, U16.1 (IN-3)
- new net: R89.2, U16.12 (IN+1)
- new net: R94.2, U16.11 (IN-1)
- new net: R96.2, U16.14 (IN-2)
- new net: R95.2, U16.15 (IN+2)
- new net: R97.2, U16.2 (IN+3)
- new net +3V3_MCU: C109.1, U16.4 (VS)
- new net SUP_3V3_PL: C60.1, C62.1, C87.1, L5.2, R39.1, R92.1, R95.1
- new net SUP_5V_PL: C59.1, C61.1, C86.1, L4.2, R37.1, R89.1, R91.1
- new net SUP_VARI_PL: C101.1, C102.1, C75.1, C76.1, C77.1, C88.1, R53.2, R93.1, R97.1, U12.12 (OUT)
- no-connect marks 1 -> 5
Other:
- note added: "MP28167 is at 0x60"
- note added: "Tie A0 → GND for address 0x40"
- note added: "WRITE THIS IN DESIGN REPORT"
- note removed: "10UF FOR DEV"
- note removed: "Enable rising threshold VEN_RISE = 1.21-1.28 V, falling VEN_FALL = 1.1-1.17 V EN pull-up current Ip = 0.7 µA, hysteresis current Ih = 1.4 µA EN absolute max = 6 V (recommended ≤ 5.5 V)"
- note removed: "PLACEHOLDER W 10UF FOR DEV"
- note removed: "PROBING"
- note removed: "RC-staggered enables (shared divider, but different C_EN - smallest cap on 1V2 so it ramps first, larger on 3V3/5V)"
- note removed: "THESE MUST BE >>0603 FOR FLIGHT - RN ONLY RATED TO 10V"
- note removed: "VARIABLE: TPS55288"
- note removed: "WURTH INDUCTOR: I_sat ≥ ~5 A and I_RMS ≥ 3 A with low DCR"
- moved on the sheet: C28, C29, C30, C31, C32, C33, C34, C35, C36, C37, C38, C39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

Commit message: pc104 outline, nearly done with layout, managed to keep it at 4 layers but the traces became quite messy; still need to do an in depth review to ensure i havent cut across any zones unknowingly; also there are still DRC errors that i need to work through - but all nets are connected !
Parts:
- removed J11, J12, J13: Conn_01x02, Connector_PinHeader_2.54mm:PinHeader_1x02_P2.54mm_Vertical, symbol Connector_Generic:Conn_01x02
- added C110: 0.1uF, Capacitor_SMD:C_0603_1608Metric, symbol Device:C_Small
- added J10, J11, J9: Conn_01x06, CustomFootprints:Molex_Pico-Lock_504050-0691_1x06-1MP_P1.50mm_Horizontal, symbol Connector_Generic:Conn_01x06
- added R128, R129, R130, R131, R132, R133, R134, R135, R136, R137, R57, R58: 0R, Resistor_SMD:R_0603_1608Metric, symbol Device:R_Small
- L1, L2, L3, L4, L5: value 6.8uH -> 2.2uF; footprint CustomFootprints:L_Wurth_WE-LHMI-7030 -> CustomFootprints:SRP5015TA-2R2M; MPN 74437346068 -> SRP5015TA-2R2M; PD FIXED IND 6.8UH 3.4A 60 MOHM SMD -> FIXED IND 2.2UH 4A 52 MOHM SMD
- L6: value 4.7uH -> 2.2uF; footprint CustomFootprints:L_Wurth_WE-LHMI-7050 -> CustomFootprints:SRP5015TA-2R2M; MPN 74437349047 -> SRP5015TA-2R2M; PD FIXED IND 4.7UH 5A 30.8 MOHM SMD -> FIXED IND 2.2UH 4A 52 MOHM SMD
- R22, R23, R24, R35, R36: now fitted
Connections:
- net +12V_HK: now also R128.1, R129.1, R130.1, R131.1, R57.1, R58.1; no longer C28.1, C29.1, C30.1, C31.1, C32.1, C33.1, C34.1, C35.1, C36.1, R45.1, R47.1, R49.1, U6.3 (VIN), U7.3 (VIN), U8.3 (VIN)
- net +12V_PL: now also R132.1, R133.1, R134.1, R135.1, R136.1, R137.1; no longer C49.1, C50.1, C51.1, C52.1, C53.1, C54.1, C68.1, C69.1, C70.1, U10.3 (VIN), U12.1 (IN), U9.3 (VIN)
- net +3V3_MCU: now also U16.16 (VPU), C110.1
- net +3V3_PL: now also J10.1 (Pin_1), J10.2 (Pin_2), J10.3 (Pin_3)
- net +5V_PL: now also J9.1 (Pin_1), J9.2 (Pin_2), J9.3 (Pin_3)
- net +VARI_PL: now also J11.1 (Pin_1), J11.2 (Pin_2), J11.3 (Pin_3)
- net GND: now also C110.2, J10.4 (Pin_4), J10.5 (Pin_5), J10.6 (Pin_6), J11.4 (Pin_4), J11.5 (Pin_5), J11.6 (Pin_6), J9.4 (Pin_4), J9.5 (Pin_5), J9.6 (Pin_6)
- net +VARI_ALT: now reaches U12.4 (ALT)
- new net: C28.1, C31.1, C34.1, R45.1, R57.2, R58.2, U6.3 (VIN)
- new net: C30.1, C33.1, C36.1, R130.2, R131.2, R49.1, U8.3 (VIN)
- new net: C68.1, C69.1, C70.1, R136.2, R137.2, U12.1 (IN)
- new net: C29.1, C32.1, C35.1, R128.2, R129.2, R47.1, U7.3 (VIN)
- new net: C50.1, C52.1, C54.1, R134.2, R135.2, U10.3 (VIN)
- new net: C49.1, C51.1, C53.1, R132.2, R133.2, U9.3 (VIN)
- no-connect marks 5 -> 4
Other:
- note added: "Firmware sequence for U12 (I²C 0x60) Drive +VARI_EN high. The chip starts at its defaults: 500 kHz, 3.5 A limit, and the output voltage set by your FB divider. That state is safe for the inductor. Immediately write CTL1 (0x04) bit D7 = 0. With the EN pin high, this bit takes over and turns the converter off while I²C stays alive. Use read-modify-write, not a hardcoded byte. Write IOUT_LIM (0x03) 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"
- note added: "RISK::: When the eFuse is off, U12 has no power but still sits on POWER_SDA/SCL. If its SDA/SCL pins clamp the bus while unpowered, the INA3221 becomes unreachable. Bench-test this with the eFuse off."
- note added: "Using SRP5015TA, MUST CAP VARI AT ABOUT 2A IN FW VIA IOUT_LIM. this keeps inductor current near 3A (sat)"
- note added: "picolock"
- moved on the sheet: C101, C102, C28, C29, C30, C31, C32, C33, C34, C35, C36, C37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
